Commit message: changes in arm_description

File: kalman_arm_moveit_config/urdf/arm_description.urdf.xacro (robot description, xacro)
@@ -154,4 +154,11 @@
         <origin rpy="0 0 0" xyz="0 0 ${link_5_length/2}"/>
     </joint>
+    <link name="d435_arm">
+    </link>
+    <joint name="joint5_camera", type="fixed">
+        <parent link="link5">
+        <child  link="d435_arm">
+        <origin rpy="0 0 0" xyz="0 0 0.1">
+    </joint>
     <link name="link5_ext">
         <visual>

Commit message: fixes

File: kalman_arm_moveit_config/urdf/arm_description.urdf.xacro (robot description, xacro)
@@ -156,8 +156,8 @@
     <link name="d435_arm">
     </link>
-    <joint name="joint5_camera", type="fixed">
-        <parent link="link5">
-        <child  link="d435_arm">
-        <origin rpy="0 0 0" xyz="0 0 0.1">
+    <joint name="joint5_camera" type="fixed">
+        <parent link="link5"/>
+        <child  link="d435_arm"/>
+        <origin rpy="0 0 0" xyz="0 0 0.1"/>
     </joint>
     <link name="link5_ext">

Commit message: maybe works

File: kalman_arm_moveit_config/urdf/arm_description.urdf.xacro (robot description, xacro)
@@ -157,7 +157,7 @@
     </link>
     <joint name="joint5_camera" type="fixed">
-        <parent link="link5"/>
+        <parent link="ee"/>
         <child  link="d435_arm"/>
-        <origin rpy="0 0 0" xyz="0 0 0.1"/>
+        <origin rpy="1.57 0 1.57" xyz="-0.2 0 0.0"/>
     </joint>
     <link name="link5_ext">

Commit message: some changes

File: kalman_arm_moveit_config/urdf/arm_description.urdf.xacro (robot description, xacro)
@@ -159,5 +159,5 @@
         <parent link="ee"/>
         <child  link="d435_arm"/>
-        <origin rpy="1.57 0 1.57" xyz="-0.2 0 0.0"/>
+        <origin rpy="1.80 0 1.57" xyz="-0.2 0 0.07"/>
     </joint>
     <link name="link5_ext">
